File: hardware/dbfob.kicad_sch (KiCad schematic)
At the start: 17 parts, among them J1 PROG, SW1 measure, U1 CH32V003F4P6

Commit message: hardware: dim LED bar, D4 doubles as ambient light sensor
Resistors 2.2k (1k for the dimmer yellow-green) cap the LEDs at
~0.45-1 mA; a club is dark and the bar should not light the room.
D4's cathode moves from GND to PC2 so the red LED can be reverse-biased
and timed as a light sensor: auto-dim indoors, brighter in daylight,
no extra part. Rerouted: DRC/parity clean, CPL check passes.

Co-Authored-By: Claude Opus 5.5 <noreply@anthropic.com>
Parts:
- R4: value 220 -> 1k; LCSC C22962 -> C21190
- R5, R6, R7: value 470 -> 2.2k; LCSC C23179 -> C4190
Connections:
- net GND: no longer D4.1 (K)
- net LED_R_K: now reaches U1.12 (PC2)
- net LED_R_K: now also D4.1 (K)
- no-connect marks 8 -> 7
Other:
- note added: "LEDs on timer channels for PWM: D1 PD3 T2C2, D2 PD2 T1C1, D3 PC4 T1C4, D4 PC3 T1C3. D4 cathode on PC2 = ambient light sense."
- note removed: "LEDs on timer channels for PWM: D1 PD3 T2C2, D2 PD2 T1C1, D3 PC4 T1C4, D4 PC3 T1C3."
Changed lines of the file:
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@@
 		(instances (project "dbfob" (path "/058019d1-3f91-5e5f-9605-7efe8396e2b2" (reference "D4") (unit 1))))
 	)
-	(label "GND"
+	(label "LED_R_K"
 		(at 134.62 64.77 270)
 		(fields_autoplaced yes)
@@
 			(effects (font (size 1.27 1.27)))
 		)
-		(property "Value" "220"
+		(property "Value" "1k"
 			(at 48.72 46.64 0)
 			(effects (font (size 1.27 1.27)))
@@
 			(effects (font (size 1.27 1.27)) (hide yes))
 		)
-		(property "LCSC" "C22962"
+		(property "LCSC" "C21190"
 			(at 45.72 40.64 0)
 			(effects (font (size 1.27 1.27)) (hide yes))
@@
 			(effects (font (size 1.27 1.27)))
 		)
-		(property "Value" "470"
+		(property "Value" "2.2k"
 			(at 79.2 46.64 0)
 			(effects (font (size 1.27 1.27)))
@@
 			(effects (font (size 1.27 1.27)) (hide yes))
 		)
-		(property "LCSC" "C23179"
+		(property "LCSC" "C4190"
 			(at 76.2 40.64 0)
 			(effects (font (size 1.27 1.27)) (hide yes))
@@
 			(effects (font (size 1.27 1.27)))
 		)
-		(property "Value" "470"
+		(property "Value" "2.2k"
 			(at 107.14 46.64 0)
 			(effects (font (size 1.27 1.27)))
@@
 			(effects (font (size 1.27 1.27)) (hide yes))
 		)
-		(property "LCSC" "C23179"
+		(property "LCSC" "C4190"
 			(at 104.14 40.64 0)
 			(effects (font (size 1.27 1.27)) (hide yes))
@@
 			(effects (font (size 1.27 1.27)))
 		)
-		(property "Value" "470"
+		(property "Value" "2.2k"
 			(at 137.62 46.64 0)
 			(effects (font (size 1.27 1.27)))
@@
 			(effects (font (size 1.27 1.27)) (hide yes))
 		)
-		(property "LCSC" "C23179"
+		(property "LCSC" "C4190"
 			(at 134.62 40.64 0)
 			(effects (font (size 1.27 1.27)) (hide yes))
@@
 		(effects (font (size 1.27 1.27)) (justify right bottom))
 	)
+	(label "LED_R_K"
+		(at 116.84 86.36 180)
+		(fields_autoplaced yes)
+		(effects (font (size 1.27 1.27)) (justify right bottom))
+	)
 	(label "SWIO"
 		(at 137.16 83.82 0)
@@
 	(no_connect
 		(at 116.84 83.82)
-	)
-	(no_connect
-		(at 116.84 86.36)
 	)
 	(wire
@@
 		(effects (font (size 1.5 1.5)) (justify left bottom))
 	)
-	(text "LEDs on timer channels for PWM: D1 PD3 T2C2, D2 PD2 T1C1, D3 PC4 T1C4, D4 PC3 T1C3."
+	(text "LEDs on timer channels for PWM: D1 PD3 T2C2, D2 PD2 T1C1, D3 PC4 T1C4, D4 PC3 T1C3. D4 cathode on PC2 = ambient light sense."
 		(exclude_from_sim no)
 		(at 20 180 0)

Commit message: Address hardware audit: clock plan, claims, power, release gates
- PDM clock 1.024 MHz sat between the IM69D130's specified bands and
  cannot be divided from 48 MHz; now 1.5 MHz (48/32 or 24/16),
  decimated by 64 to 23,437.5 samples/s.
- Bands restated as levels at the ear with allowance times from the
  stated curve (96 dBA = 38 min, not an hour); the plugs LED is a
  conditional estimate, not a safety verdict. Silk legend updated.
- Power: unsupported 10-15% capacity claim withdrawn; qualification
  plan, under-load cutoff, standby budget (V003 7.6 uA ~ 67 mAh/yr).
- Programming: remove the cell first (J1 pin 1 is the cell's +);
  back silk, schematic note and README say so.
- make_pcb.py and fab.py now fail on any ERC/DRC/parity finding beyond
  the documented ones; fab.py stages outputs and publishes only after
  check_cpl.py passes, which now also checks BOM/CPL membership,
  duplicates and layer.
- Mic lifecycle recorded as unresolved (DigiKey: Active).

Co-Authored-By: Claude Opus 5.5 <noreply@anthropic.com>
Other:
- note added: "D4 cathode on PC2 = ambient light sense."
- note added: "LED PWM: D1 PD3 T2C2, D2 PD2 T1C1, D3 PC4 T1C4, D4 PC3 T1C3."
- note added: "Mic powered from PC6 only while measuring."
- note added: "PDM mic on SPI1: PC5 SCK -> CLK at 1.5 MHz, PC7 MISO <- DATA."
- note added: "Remove the cell before programming through J1."
- note added: "U1 fitted CH32V003F4P6; CH32V002/V006 drop-in."
- note removed: "LEDs on timer channels for PWM: D1 PD3 T2C2, D2 PD2 T1C1, D3 PC4 T1C4, D4 PC3 T1C3. D4 cathode on PC2 = ambient light sense."
- note removed: "PDM mic on SPI: PC5 SCK -> CLK, PC7 MISO <- DATA, mic powered from PC6 only while measuring."
- note removed: "U1 fitted as CH32V003F4P6 (in stock); CH32V002F4P6 / CH32V006F8P6 are drop-in on this footprint."
Changed lines of the file:
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@@
 	(symbol
 		(lib_id "power:PWR_FLAG")
-		(at 71.12 149.86 0)
+		(at 109.22 139.7 0)
 		(unit 1)
 		(exclude_from_sim no)
@@
 		(dnp no)
 		(property "Reference" "#FLG02"
-			(at 74.12 143.86 0)
+			(at 112.22 133.7 0)
 			(effects (font (size 1.27 1.27)) (hide yes))
 		)
 		(property "Value" "PWR_FLAG"
-			(at 74.12 155.86 0)
+			(at 112.22 145.7 0)
 			(effects (font (size 1.27 1.27)) (hide yes))
 		)
 		(property "Footprint" ""
-			(at 71.12 149.86 0)
+			(at 109.22 139.7 0)
 			(effects (font (size 1.27 1.27)) (hide yes))
 		)
 		(property "Datasheet" ""
-			(at 71.12 149.86 0)
+			(at 109.22 139.7 0)
 			(effects (font (size 1.27 1.27)) (hide yes))
 		)
@@
 	)
 	(label "GND"
-		(at 71.12 149.86 270)
+		(at 109.22 139.7 270)
 		(fields_autoplaced yes)
 		(effects (font (size 1.27 1.27)) (justify right bottom))
@@
 		(effects (font (size 2.5 2.5)) (justify left bottom))
 	)
-	(text "PDM mic on SPI: PC5 SCK -> CLK, PC7 MISO <- DATA, mic powered from PC6 only while measuring."
+	(text "PDM mic on SPI1: PC5 SCK -> CLK at 1.5 MHz, PC7 MISO <- DATA."
 		(exclude_from_sim no)
-		(at 20 175 0)
+		(at 20 150 0)
 		(effects (font (size 1.5 1.5)) (justify left bottom))
 	)
-	(text "LEDs on timer channels for PWM: D1 PD3 T2C2, D2 PD2 T1C1, D3 PC4 T1C4, D4 PC3 T1C3. D4 cathode on PC2 = ambient light sense."
+	(text "Mic powered from PC6 only while measuring."
 		(exclude_from_sim no)
-		(at 20 180 0)
+		(at 20 154 0)
 		(effects (font (size 1.5 1.5)) (justify left bottom))
 	)
-	(text "U1 fitted as CH32V003F4P6 (in stock); CH32V002F4P6 / CH32V006F8P6 are drop-in on this footprint."
+	(text "LED PWM: D1 PD3 T2C2, D2 PD2 T1C1, D3 PC4 T1C4, D4 PC3 T1C3."
 		(exclude_from_sim no)
-		(at 20 185 0)
+		(at 20 158 0)
 		(effects (font (size 1.5 1.5)) (justify left bottom))
 	)
+	(text "D4 cathode on PC2 = ambient light sense."
+		(exclude_from_sim no)
+		(at 20 162 0)
+		(effects (font (size 1.5 1.5)) (justify left bottom))
+	)
+	(text "U1 fitted CH32V003F4P6; CH32V002/V006 drop-in."
+		(exclude_from_sim no)
+		(at 20 166 0)
+		(effects (font (size 1.5 1.5)) (justify left bottom))
+	)
+	(text "Remove the cell before programming through J1."
+		(exclude_from_sim no)
+		(at 20 170 0)
+		(effects (font (size 1.5 1.5)) (justify left bottom))
+	)
